File: Hardware/KiCAD/AltoidsSmall/AltoidsSmall.kicad_pcb (KiCad board)
At the start: 4 copper layers, 55 x 35 mm, 42 parts, among them J1 Conn_01x10_Male, J2 Conn_01x10_Male, J3 Conn_01x03_Male, J4 Conn_01x03_Male, J5 Conn_01x06_Male, SW1 SW_Push, SW2 SW_Push, U1 SC662K-3.3V, U2 STM32F103C8Tx, U3 FT230XQ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

Commit message: Added CAMFILES
Parts:
- added C16: 1uF, Capacitor_SMD:C_0603_1608Metric_Pad1.05x0.95mm_HandSolder, F.Cu at (161.5, 128.1)
- added C17: 1uF, Capacitor_SMD:C_0603_1608Metric_Pad1.05x0.95mm_HandSolder, F.Cu at (156.4, 128.0)
- added C18: 18pF, Capacitor_SMD:C_0603_1608Metric_Pad1.05x0.95mm_HandSolder, F.Cu at (144.3, 125.9)
- added C19: 18pF, Capacitor_SMD:C_0603_1608Metric_Pad1.05x0.95mm_HandSolder, F.Cu at (144.1, 120.8)
- added FB1: Ferrite_Bead_Small, Capacitor_SMD:C_0805_2012Metric, F.Cu at (161.6, 132.5)
- added U6: SC662K-3.3V, Package_TO_SOT_SMD:SOT-23, F.Cu at (158.9, 128.1)
- added Y1: Crystal_GND24_Small, Crystal:Crystal_SMD_Abracon_ABM8G-4Pin_3.2x2.5mm, F.Cu at (144.3, 123.5)
- C13: footprint Capacitor_SMD:C_0603_1608Metric_Pad1.05x0.95mm_HandSolder -> Capacitor_SMD:C_0805_2012Metric
- D1, D2, D3: footprint Capacitor_SMD:C_0603_1608Metric_Pad1.05x0.95mm_HandSolder -> Diode_SMD:D_0603_1608Metric_Castellated
- moved SW2 6.12 mm to (149.2, 126.9)
- moved R5 1.59 mm to (146.9, 119.4)
- moved R3 0.58 mm to (141.7, 128.3)
- moved D1 0.58 mm to (139.9, 128.2)
Connections:
- C14 pad 1: +3V3 -> VDDA
- C15 pad 1: +3V3 -> VDDA
- R11 pad 1: +3V3 -> VDDA
- U2 pad 5: (no net) -> Net-(C18-Pad1)
- U2 pad 6: (no net) -> Net-(C19-Pad1)
- U5 pad 1: +3V3 -> VDDA
Routing:
- net VDDA: track 0.00 -> 65.0 mm, vias 0 -> 4
- net VBUS: track 26.3 -> 38.9 mm
- net +3V3: track 46.8 -> 37.3 mm, vias 21 -> 20
- net Net-(C19-Pad1): track 0.00 -> 8.55 mm
- net Net-(C18-Pad1): track 0.00 -> 6.80 mm
- net Net-(C16-Pad1): track 0.00 -> 5.42 mm
- net /MCU/~RST: track 17.4 -> 21.9 mm
- net Net-(J2-Pad1): track 26.3 -> 29.7 mm
- net GND: track 37.2 -> 40.0 mm, vias 21 -> 28
- net Net-(R3-Pad2): track 7.68 -> 7.03 mm
