File: Hardware/KiCAD/AltoidsSmall/STM32F103.sch (KiCad schematic (older format))
At the start: 22 parts, among them J1 Conn_01x10_Male, J2 Conn_01x10_Male, J3 Conn_01x03_Male, J4 Conn_01x03_Male, SW1 SW_Push, SW2 SW_Push, U2 STM32F103C8Tx, Y1 Crystal_GND24_Small

Commit message: Added labels to pins, Added part numbers
Parts:
- C18, C19: Digikey (none) -> 13-CC0603JRNPO8BN180CT-ND
- C3, C4, C5, C7: Digikey (none) -> 1276-CL10B104KB8VPJCCT-ND
- C6, C8: Digikey (none) -> H 5600 2125 50 0001 C CNN
- D1: footprint Capacitor_SMD:C_0603_1608Metric_Pad1.05x0.95mm_HandSolder -> Diode_SMD:D_0603_1608Metric_Castellated
- R1, R2: Digikey (none) -> CR0603-FX-4991ELFCT-ND
Changed lines of the file:
@@
 F 2 "Capacitor_SMD:C_0603_1608Metric_Pad1.05x0.95mm_HandSolder" H 7775 2175 50  0001 C CNN
 F 3 "~" H 7775 2175 50  0001 C CNN
-F 4 "" H 7775 2175 50  0001 C CNN "Digikey"
+F 4 "1276-CL10B104KB8VPJCCT-ND" H 7775 2175 50  0001 C CNN "Digikey"
 F 5 "C1591" H 7775 2175 50  0001 C CNN "LCSC"
 	1    7775 2175
@@
 F 2 "Capacitor_SMD:C_0603_1608Metric_Pad1.05x0.95mm_HandSolder" H 8175 2175 50  0001 C CNN
 F 3 "~" H 8175 2175 50  0001 C CNN
-F 4 "" H 8175 2175 50  0001 C CNN "Digikey"
+F 4 "1276-CL10B104KB8VPJCCT-ND" H 8175 2175 50  0001 C CNN "Digikey"
 F 5 "C1591" H 8175 2175 50  0001 C CNN "LCSC"
 	1    8175 2175
@@
 F 2 "Capacitor_SMD:C_0603_1608Metric_Pad1.05x0.95mm_HandSolder" H 8575 2175 50  0001 C CNN
 F 3 "~" H 8575 2175 50  0001 C CNN
-F 4 "" H 8575 2175 50  0001 C CNN "Digikey"
+F 4 "1276-CL10B104KB8VPJCCT-ND" H 8575 2175 50  0001 C CNN "Digikey"
 F 5 "C1591" H 8575 2175 50  0001 C CNN "LCSC"
 	1    8575 2175
@@
 F 2 "Capacitor_SMD:C_0603_1608Metric_Pad1.05x0.95mm_HandSolder" H 9275 2175 50  0001 C CNN
 F 3 "~" H 9275 2175 50  0001 C CNN
-F 4 "" H 9275 2175 50  0001 C CNN "Digikey"
+F 4 "1276-CL10B104KB8VPJCCT-ND" H 9275 2175 50  0001 C CNN "Digikey"
 F 5 "C1591" H 9275 2175 50  0001 C CNN "LCSC"
 	1    9275 2175
@@
 F 0 "D1" V 3821 3605 50  0000 R CNN
 F 1 "LED_Small_ALT" V 3730 3605 50  0000 R CNN
-F 2 "Capacitor_SMD:C_0603_1608Metric_Pad1.05x0.95mm_HandSolder" V 3775 3675 50  0001 C CNN
+F 2 "Diode_SMD:D_0603_1608Metric_Castellated" V 3775 3675 50  0001 C CNN
 F 3 "~" V 3775 3675 50  0001 C CNN
 F 4 "" V 3775 3675 50  0001 C CNN "Digikey"
@@
 F 2 "Resistor_SMD:R_0603_1608Metric_Pad1.05x0.95mm_HandSolder" H 3200 3725 50  0001 C CNN
 F 3 "~" H 3200 3725 50  0001 C CNN
-F 4 "" H 3200 3725 50  0001 C CNN "Digikey"
+F 4 "CR0603-FX-4991ELFCT-ND" H 3200 3725 50  0001 C CNN "Digikey"
 F 5 "C441891" H 3200 3725 50  0001 C CNN "LCSC"
 	1    3200 3725
@@
 F 2 "Resistor_SMD:R_0603_1608Metric_Pad1.05x0.95mm_HandSolder" H 3000 3750 50  0001 C CNN
 F 3 "~" H 3000 3750 50  0001 C CNN
-F 4 "" H 3000 3750 50  0001 C CNN "Digikey"
+F 4 "CR0603-FX-4991ELFCT-ND" H 3000 3750 50  0001 C CNN "Digikey"
 F 5 "C441891" H 3000 3750 50  0001 C CNN "LCSC"
 	1    3000 3750
@@
 F 2 "Capacitor_SMD:C_0603_1608Metric_Pad1.05x0.95mm_HandSolder" H 8975 2175 50  0001 C CNN
 F 3 "~" H 8975 2175 50  0001 C CNN
-F 4 "" H 8975 2175 50  0001 C CNN "Digikey"
+F 4 "H 5600 2125 50  0001 C CNN" H 8975 2175 50  0001 C CNN "Digikey"
 F 5 "" H 8975 2175 50  0001 C CNN "LCSC"
 	1    8975 2175
@@
 F 2 "Capacitor_SMD:C_0603_1608Metric_Pad1.05x0.95mm_HandSolder" H 9675 2175 50  0001 C CNN
 F 3 "~" H 9675 2175 50  0001 C CNN
-F 4 "" H 9675 2175 50  0001 C CNN "Digikey"
+F 4 "H 5600 2125 50  0001 C CNN" H 9675 2175 50  0001 C CNN "Digikey"
 F 5 "" H 9675 2175 50  0001 C CNN "LCSC"
 	1    9675 2175
@@
 F 2 "Capacitor_SMD:C_0603_1608Metric_Pad1.05x0.95mm_HandSolder" H 3275 3075 50  0001 C CNN
 F 3 "~" H 3275 3075 50  0001 C CNN
+F 4 "13-CC0603JRNPO8BN180CT-ND" H 3275 3075 50  0001 C CNN "Digikey"
 	1    3275 3075
 	1    0    0    -1
@@
 F 2 "Capacitor_SMD:C_0603_1608Metric_Pad1.05x0.95mm_HandSolder" H 3575 3075 50  0001 C CNN
 F 3 "~" H 3575 3075 50  0001 C CNN
+F 4 "13-CC0603JRNPO8BN180CT-ND" H 3575 3075 50  0001 C CNN "Digikey"
 	1    3575 3075
 	1    0    0    -1
