File: Hardware/KiCAD/AltoidsSmall/_autosave-MCP4728.sch (KiCad schematic (older format))
At the start: 6 parts, among them J5 Conn_01x06_Male, U5 MCP4728

Commit message: Added labels to pins, Added part numbers
Parts:
- C14: Digikey (none) -> 1276-CL10B104KB8VPJCCT-ND
- C15: Digikey (none) -> H 5600 2125 50 0001 C CNN
- R11: Digikey (none) -> RMCF0603JT100KCT-ND
- U5: Digikey (none) -> MCP4728A0T-E/UNCT-ND
Changed lines of the file:
@@
 F 2 "Package_SO:MSOP-10_3x3mm_P0.5mm" H 5825 3000 50  0001 C CNN
 F 3 "http://ww1.microchip.com/downloads/en/DeviceDoc/22187E.pdf" H 5825 3850 50  0001 C CNN
+F 4 "MCP4728A0T-E/UNCT-ND" H 5825 3600 50  0001 C CNN "Digikey"
 	1    5825 3600
 	1    0    0    -1
@@
 F 2 "Resistor_SMD:R_0603_1608Metric_Pad1.05x0.95mm_HandSolder" H 4125 3675 50  0001 C CNN
 F 3 "~" H 4125 3675 50  0001 C CNN
-F 4 "" H 4125 3675 50  0001 C CNN "Digikey"
+F 4 "RMCF0603JT100KCT-ND" H 4125 3675 50  0001 C CNN "Digikey"
 F 5 "C441891" H 4125 3675 50  0001 C CNN "LCSC"
 	1    4125 3675
@@
 F 2 "Capacitor_SMD:C_0603_1608Metric_Pad1.05x0.95mm_HandSolder" H 5200 3175 50  0001 C CNN
 F 3 "~" H 5200 3175 50  0001 C CNN
-F 4 "" H 5200 3175 50  0001 C CNN "Digikey"
+F 4 "1276-CL10B104KB8VPJCCT-ND" H 5200 3175 50  0001 C CNN "Digikey"
 F 5 "" H 5200 3175 50  0001 C CNN "LCSC"
 	1    5200 3175
@@
 F 2 "Capacitor_SMD:C_0603_1608Metric_Pad1.05x0.95mm_HandSolder" H 5600 3175 50  0001 C CNN
 F 3 "~" H 5600 3175 50  0001 C CNN
-F 4 "" H 5600 3175 50  0001 C CNN "Digikey"
+F 4 "H 5600 2125 50  0001 C CNN" H 5600 3175 50  0001 C CNN "Digikey"
 F 5 "" H 5600 3175 50  0001 C CNN "LCSC"
 	1    5600 3175
