File: Hardware/KiCAD/AltoidsSmall/_autosave-USB2FTDI.sch (KiCad schematic (older format))
At the start: 13 parts, among them U3 FT230XQ

Commit message: Added labels to pins, Added part numbers
Parts:
- C10, C11: Digikey (none) -> 311-4037-1-ND
- C12, C9: Digikey (none) -> 1276-CL10B104KB8VPJCCT-ND
- D2, D3: Digikey (none) -> 475-1276-1-ND
- R7, R8: Digikey (none) -> RR08Q27DCT-ND
- U3: Digikey (none) -> 768-1130-1-ND
Changed lines of the file:
@@
 F 2 "Diode_SMD:D_0603_1608Metric_Castellated" V 7000 3700 50  0001 C CNN
 F 3 "~" V 7000 3700 50  0001 C CNN
+F 4 "475-1276-1-ND" V 7000 3700 50  0001 C CNN "Digikey"
 	1    7000 3700
 	0    -1   -1   0
@@
 F 2 "Resistor_SMD:R_0603_1608Metric_Pad1.05x0.95mm_HandSolder" H 4625 3500 50  0001 C CNN
 F 3 "~" H 4625 3500 50  0001 C CNN
+F 4 "RR08Q27DCT-ND" V 4625 3500 50  0001 C CNN "Digikey"
 	1    4625 3500
 	0    1    1    0
@@
 F 2 "Resistor_SMD:R_0603_1608Metric_Pad1.05x0.95mm_HandSolder" H 4625 3600 50  0001 C CNN
 F 3 "~" H 4625 3600 50  0001 C CNN
+F 4 "RR08Q27DCT-ND" V 4625 3600 50  0001 C CNN "Digikey"
 	1    4625 3600
 	0    1    1    0
@@
 F 2 "Capacitor_SMD:C_0603_1608Metric_Pad1.05x0.95mm_HandSolder" H 4275 4125 50  0001 C CNN
 F 3 "~" H 4275 4125 50  0001 C CNN
+F 4 "311-4037-1-ND" H 4275 4125 50  0001 C CNN "Digikey"
 	1    4275 4125
 	1    0    0    -1
@@
 F 2 "Capacitor_SMD:C_0603_1608Metric_Pad1.05x0.95mm_HandSolder" H 4425 4125 50  0001 C CNN
 F 3 "~" H 4425 4125 50  0001 C CNN
+F 4 "311-4037-1-ND" H 4425 4125 50  0001 C CNN "Digikey"
 	1    4425 4125
 	1    0    0    -1
@@
 F 2 "Capacitor_SMD:C_0603_1608Metric_Pad1.05x0.95mm_HandSolder" H 7175 2625 50  0001 C CNN
 F 3 "~" H 7175 2625 50  0001 C CNN
+F 4 "1276-CL10B104KB8VPJCCT-ND" H 7175 2625 50  0001 C CNN "Digikey"
 	1    7175 2625
 	1    0    0    -1
@@
 F 2 "Capacitor_SMD:C_0603_1608Metric_Pad1.05x0.95mm_HandSolder" H 3450 3300 50  0001 C CNN
 F 3 "~" H 3450 3300 50  0001 C CNN
+F 4 "1276-CL10B104KB8VPJCCT-ND" H 3450 3300 50  0001 C CNN "Digikey"
 	1    3450 3300
 	1    0    0    -1
@@
 F 2 "Diode_SMD:D_0603_1608Metric_Castellated" V 6475 3700 50  0001 C CNN
 F 3 "~" V 6475 3700 50  0001 C CNN
+F 4 "475-1276-1-ND" V 6475 3700 50  0001 C CNN "Digikey"
 	1    6475 3700
 	0    -1   -1   0
@@
 F 2 "Package_DFN_QFN:QFN-16-1EP_4x4mm_P0.65mm_EP2.1x2.1mm" H 6850 3000 50  0001 C CNN
 F 3 "https://www.ftdichip.com/Support/Documents/DataSheets/ICs/DS_FT230X.pdf" H 5500 3600 50  0001 C CNN
+F 4 "768-1130-1-ND" H 5500 3600 50  0001 C CNN "Digikey"
 	1    5500 3600
 	1    0    0    -1
